Commit message: added tutorial_2 files

File: platforms/robotiq/robotiq_description/urdf/robotiq_85_gripper.urdf.xacro (robot description, xacro)
@@ -32,5 +32,6 @@
       <axis xyz="0 0 1"/>
       <origin rpy="${pi} 0.0 0.0" xyz="0.05490451627 0.03060114443 0.0"/>
-      <limit lower="0.0" upper="0.80285" velocity="10.5" effort="0.1"/>
+      <!-- <limit lower="0.0" upper="0.80285" velocity="10.5" effort="0.1"/> -->
+      <limit lower="-0.2" upper="1." velocity="10.5" effort="0.1"/>
       <dynamics damping="0.1" friction="0.0"/>
     </joint>
@@ -40,5 +41,6 @@
       <axis xyz="0 0 1"/>
       <origin rpy="0.0 0.0 0.0" xyz="0.05490451627 -0.03060114443 0.0"/>
-      <limit lower="0.0" upper="0.80285" velocity="10.5" effort="0.1"/>
+      <!-- <limit lower="0.0" upper="0.80285" velocity="10.5" effort="0.1"/> -->
+      <limit lower="-0.2" upper="1." velocity="10.5" effort="0.1"/>
       <mimic joint="${prefix}robotiq_85_left_knuckle_joint"/>
     </joint>
